Commit message: camera and code for recognizing the green ball added

File: src/SLAM_packages-main/slam_gmapping/gmapping/urdf/robot2_laser.xacro (robot description, xacro)
@@ -139,7 +139,35 @@
   <joint name="hokuyo_joint" type="fixed">
 	    <axis xyz="0 1 0" />
-	    <origin xyz="0.28 0 0.05" rpy="0 0 0"/>
+	    <origin xyz="0.28 0.035 0.05" rpy="0 0 0"/>
 	    <parent link="link_chassis"/>
 	    <child link="hokuyo_link"/>
 	 </joint>
+ <link name="camera_link">
+	    <collision>
+	      <origin xyz="0 0 0.025" rpy="0 0 0"/>
+	      <geometry>
+		<box size="0.05 0.05 0.05"/>
+	      </geometry>
+	    </collision>
+	    <visual>
+	      <origin xyz="0 0 0.025" rpy="0 0 0"/>
+	      <geometry>
+		<box size="0.05 0.05 0.05"/>
+	      </geometry>
+	      <material name="blue">
+		<color rgba="1 0 0 1"/>
+	      </material>
+	    </visual>
+	    <inertial>
+	      <mass value="1e-5" />
+	      <origin xyz="0 0 0.005" rpy="0 0 0"/>
+	      <inertia ixx="1e-6" ixy="0" ixz="0" iyy="1e-6" iyz="0" izz="1e-6" />
+	    </inertial>
+  </link>
+  <joint name="camera_joint" type="fixed">
+	    <axis xyz="0 1 0" />
+	    <origin xyz="0.28 -0.035 0.05" rpy="0 0 0"/>
+	    <parent link="link_chassis"/>
+	    <child link="camera_link"/>
+	 </joint>
 </robot>

Commit message: track sub_state and yaml file for parameter server added

File: src/SLAM_packages-main/slam_gmapping/gmapping/urdf/robot2_laser.xacro (robot description, xacro)
@@ -139,5 +139,5 @@
   <joint name="hokuyo_joint" type="fixed">
 	    <axis xyz="0 1 0" />
-	    <origin xyz="0.28 0.035 0.05" rpy="0 0 0"/>
+	    <origin xyz="0.28 0.055 0.05" rpy="0 0 0"/>
 	    <parent link="link_chassis"/>
 	    <child link="hokuyo_link"/>
@@ -167,5 +167,5 @@
   <joint name="camera_joint" type="fixed">
 	    <axis xyz="0 1 0" />
-	    <origin xyz="0.28 -0.035 0.05" rpy="0 0 0"/>
+	    <origin xyz="0.28 -0.01 0.05" rpy="0 0 0"/>
 	    <parent link="link_chassis"/>
 	    <child link="camera_link"/>
